File: board/ppgimp.brd (EAGLE design)
At the start: 160 x 100 mm, 11 parts, among them J1 VDD, J2 GND, J3 SPI, J4 I_Test, J5 R_test, U1 LM334Z/NOPB, U2 AD8400ARZ1, U3 AD8400ARZ10, U4 AD8400ARZ10

Commit message: do more research hook up ad5399
Parts:
- added C1: 0.1uF, scono:0603-CAP
- added C2: 10uF, scono:0603-CAP
- added FB1: (no value), scono:0603-FERR
- added J6: SDA, scono:1X02
- added R2, R3: (no value), scono:R0603
- added RFB: 1M, scono:R0603
- added U5: AD5933YRSZ, scono:RS_16
- added U6: ADG1609, scono:RU_16
Connections:
- new net AGND: FB1.1, U5.13, U5.14
- new net N$2: RFB.2, U5.4
- new net SCL: J6.2, R3.1, U5.16
- new net SDA: J6.1, R2.1, U5.15
- new net VIN: RFB.1, U5.5
- new net VOUT: U5.6
- net GND: now also C1.1, C2.1, FB1.2, U5.12
- net VDD: now also C1.2, C2.2, R2.2, R3.2, U5.10, U5.11, U5.9, U6.14
Routing:
- net GND: track 0.00 -> 13.3 mm
- net VDD: track 53.2 -> 40.7 mm, vias 3 -> 7
- net SCL: track 0.00 -> 9.84 mm
- net SDA: track 0.00 -> 7.66 mm
- net AGND: track 0.00 -> 7.42 mm
- net R: track 27.6 -> 23.3 mm, vias 2 -> 1
- net N$2: track 0.00 -> 3.00 mm
- net VIN: track 0.00 -> 2.58 mm
- added copper zone on layer 16, net VDD

Commit message: finish up test board
Parts:
- added C3, C4: 1uF, scono:0603-CAP
- added J7: SEL, scono:1X02
- added R4: 510K, scono:R0603
- added R5: 200K, scono:R0603
- added R6: 100K, scono:R0603
- R2, R3: value (none) -> 10K
- moved U6 0.50 mm to (28.0, 5.50), turned to 180 degrees
- renumbered U$1 to D1
Connections:
- new net N$10: C3.2, U6.11
- new net N$11: C4.1, R6.1, U6.7
- new net N$12: C4.2, R6.2, U6.10
- new net N$3: J7.1, U6.16
- new net N$4: J7.2, U6.1
- new net N$5: R4.2, U6.4
- new net N$6: R4.1, U6.13
- new net N$7: R5.2, U6.5
- new net N$8: R5.1, U6.12
- new net N$9: C3.1, U6.6
- net GND: now also U6.15, U6.3
- net VDD: now also U6.2
- net VIN: now also U6.8
- net VOUT: now also U6.9
Routing:
- net N$11: track 0.00 -> 13.2 mm
- net VOUT: track 0.00 -> 12.3 mm, vias 0 -> 2
- net N$5: track 0.00 -> 11.1 mm, vias 0 -> 2
- net N$12: track 0.00 -> 10.8 mm
- net N$9: track 0.00 -> 10.6 mm, vias 0 -> 2
- net N$7: track 0.00 -> 8.96 mm, vias 0 -> 2
- net N$4: track 0.00 -> 8.49 mm, vias 0 -> 1
- net N$3: track 0.00 -> 6.17 mm
- net N$10: track 0.00 -> 5.87 mm
- net N$8: track 0.00 -> 5.02 mm
- net VIN: track 2.58 -> 5.92 mm
- net N$6: track 0.00 -> 2.90 mm
- net VDD: track 40.7 -> 43.5 mm, vias 7 -> 8
Other:
- board size 160 x 100 mm -> 32.5 x 29 mm
- board text added: "Arias Research Group Bioimpedence PPG S. Ono Sp'19"

Commit message: finalize prototype
Parts:
- added C5: 0.1uF, scono:0603-CAP
- added C6: 10uF, scono:0603-CAP
- J6: value SDA -> I2C
- U5: value AD5933YRSZ -> AD5933
- moved J7 0.50 mm to (20.0, 2.50)
Connections:
- net GND: now also C5.1, C6.1
- net VDD: now also C5.2, C6.2
Routing:
- net GND: track 13.1 -> 20.8 mm, vias 0 -> 3
- net VDD: track 43.5 -> 47.6 mm
