File: board/ppgimp.sch (EAGLE design)
At the start: 0 parts

Commit message: get current source testing done
Parts:
- added J1: VDD, scono:CONN_02
- added J2: GND, scono:CONN_02
- added J3: SPI, scono:CONN_04
- added J4: I_Test, scono:CONN_02
- added J5: R_test, scono:CONN_02
- added R1: (no value), scono:POT-3PIN
- added U$1: 1N457, scono:1N457
- added U1: LM334Z/NOPB, scono:LM334Z/NOPB
- added U2: AD8400ARZ1, scono:AD8400ARZ1
- added U3, U4: AD8400ARZ10, scono:AD8400ARZ10
Connections:
- new net 10KCS: J3.4, U3.!CS, U4.!CS
- new net 1KCS: J3.3, U2.!
- new net A1: J5.1, U4.A1
- new net GND: J2.1, J2.2, J4.2, U2.GND, U3.GND, U4.GND
- new net I_OUT: R1.2, U$1.N, U3.W1
- new net MOSI: J3.2, U2.SDI, U3.SDI, U4.SDI
- new net N$1: J4.1, R1.3
- new net R: U1.R, U2.A1, U3.A1
- new net SCLK: J3.1, U2.CLK, U3.CLK, U4.CLK
- new net V-: U$1.P, U1.V-, U2.W1
- new net VDD: J1.1, J1.2, U1.V+, U2.VDD, U3.VDD, U4.VDD
- new net W1: J5.2, U4.W1

Commit message: do more research hook up ad5399
Parts:
- added C1: 0.1uF, scono:CAP0603-CAP
- added C2: 10uF, scono:CAP0603-CAP
- added FB1: (no value), scono:FERRITE
- added J6: SDA, scono:CONN_02
- added R2, R3: (no value), scono:R-US_R0603
- added RFB: 1M, scono:R-US_R0603
- added U5: AD5933YRSZ, scono:AD5933YRSZ
- added U6: ADG1609, scono:ADG1609
Connections:
- new net AGND: FB1.P$1, U5.AGND1, U5.AGND2
- new net N$2: RFB.2, U5.RFB
- new net SCL: J6.2, R3.1, U5.SCL
- new net SDA: J6.1, R2.1, U5.SDA
- new net VIN: RFB.1, U5.VIN
- new net VOUT: U5.VOUT
- net GND: now also C1.1, C2.1, FB1.P$2, U5.DGND
- net VDD: now also C1.2, C2.2, R2.2, R3.2, U5.AVDD1, U5.AVDD2, U5.DVDD, U6.VDD
Changed lines of the file:
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@@
 <?xml version="1.0" encoding="utf-8"?>
 <!DOCTYPE eagle SYSTEM "eagle.dtd">
-<eagle version="9.3.0">
+<eagle version="9.3.1">
 <drawing>
 <settings>
@@
 <setting verticaltext="up"/>
 </settings>
-<grid distance="0.1" unitdist="inch" unit="inch" style="dots" multiple="1" display="yes" altdistance="0.01" altunitdist="inch" altunit="inch"/>
+<grid distance="0.1" unitdist="inch" unit="inch" style="lines" multiple="1" display="no" altdistance="0.01" altunitdist="inch" altunit="inch"/>
 <layers>
 <layer number="1" name="Top" color="4" fill="1" visible="no" active="no"/>
@@
 <attribute name="SUBSYSTEM_NAME" value="Imepdence"/>
 </part>
+<part name="U5" library="scono" deviceset="AD5933YRSZ" device=""/>
+<part name="C1" library="scono" deviceset="CAP" device="0603-CAP" value="0.1uF"/>
+<part name="C2" library="scono" deviceset="CAP" device="0603-CAP" value="10uF"/>
+<part name="SUPPLY6" library="scono" deviceset="GND" device=""/>
+<part name="R2" library="scono" deviceset="R-US_" device="R0603"/>
+<part name="R3" library="scono" deviceset="R-US_" device="R0603"/>
+<part name="SUPPLY7" library="scono" deviceset="AGND" device=""/>
+<part name="SUPPLY8" library="scono" deviceset="GND" device=""/>
+<part name="J6" library="scono" deviceset="CONN_02" device="" package3d_urn="urn:adsk.eagle:package:38039/1" value="SDA"/>
+<part name="RFB" library="scono" deviceset="R-US_" device="R0603" value="1M"/>
+<part name="U6" library="scono" deviceset="ADG1609" device=""/>
+<part name="SUPPLY9" library="scono" deviceset="AGND" device=""/>
+<part name="SUPPLY10" library="scono" deviceset="GND" device=""/>
+<part name="FB1" library="scono" deviceset="FERRITE" device=""/>
 </parts>
 <sheets>
@@
 <attribute name="REV" x="236.22" y="6.985" size="2.7432" layer="94" font="vector"/>
 </instance>
+<instance part="U5" gate="A" x="88.9" y="132.08" smashed="yes">
+<attribute name="NAME" x="107.0356" y="141.1986" size="2.0828" layer="95" ratio="6" rot="SR0"/>
+<attribute name="VALUE" x="106.4006" y="138.6586" size="2.0828" layer="96" ratio="6" rot="SR0"/>
+</instance>
+<instance part="C1" gate="G$1" x="63.5" y="129.54" smashed="yes" rot="R90">
+<attribute name="NAME" x="61.976" y="128.27" size="1.016" layer="95" rot="R90"/>
+<attribute name="VALUE" x="66.04" y="128.27" size="1.016" layer="96" rot="R90"/>
+</instance>
+<instance part="C2" gate="G$1" x="55.88" y="129.54" smashed="yes" rot="R90">
+<attribute name="NAME" x="54.356" y="128.27" size="1.016" layer="95" rot="R90"/>
+<attribute name="VALUE" x="58.42" y="128.27" size="1.016" layer="96" rot="R90"/>
+</instance>
+<instance part="SUPPLY6" gate="GND" x="55.88" y="124.46" smashed="yes">
+<attribute name="VALUE" x="54.61" y="121.92" size="1.016" layer="96"/>
+</instance>
+<instance part="R2" gate="G$1" x="149.86" y="116.84" smashed="yes" rot="R90">
+<attribute name="NAME" x="148.59" y="111.76" size="1.016" layer="95" rot="R90"/>
+<attribute name="VALUE" x="151.13" y="111.76" size="1.016" layer="96" rot="R90" align="top-left"/>
+</instance>
+<instance part="R3" gate="G$1" x="157.48" y="114.3" smashed="yes" rot="R90">
+<attribute name="NAME" x="156.21" y="109.22" size="1.016" layer="95" rot="R90"/>
+<attribute name="VALUE" x="158.75" y="109.22" size="1.016" layer="96" rot="R90" align="top-left"/>
+</instance>
+<instance part="SUPPLY7" gate="G$1" x="137.16" y="116.84" smashed="yes" rot="R90">
+<attribute name="VALUE" x="138.684" y="115.57" size="1.016" layer="96" rot="R90" align="top-left"/>
+</instance>
+<instance part="SUPPLY8" gate="GND" x="137.16" y="121.92" smashed="yes" rot="R90">
+<attribute name="VALUE" x="139.7" y="120.65" size="1.016" layer="96" rot="R90"/>
+</instance>
+<instance part="J6" gate="G$1" x="134.62" y="99.06" smashed="yes">
+<attribute name="VALUE" x="132.08" y="94.234" size="1.778" layer="96" font="vector"/>
+<attribute name="NAME" x="132.08" y="104.648" size="1.778" layer="95" font="vector"/>
+</instance>
+<instance part="RFB" gate="G$1" x="86.36" y="109.22" smashed="yes">
+<attribute name="NAME" x="81.28" y="110.49" size="1.016" layer="95"/>
+<attribute name="VALUE" x="81.28" y="107.95" size="1.016" layer="96" align="top-left"/>
+</instance>
+<instance part="U6" gate="A" x="86.36" y="73.66" smashed="yes">
+<attribute name="NAME" x="93.98" y="81.28" size="2.0828" layer="95" ratio="6" rot="SR0" align="top-left"/>
+<attribute name="VALUE" x="116.84" y="81.28" size="2.0828" layer="96" ratio="6" rot="SR0" align="top-left"/>
+</instance>
+<instance part="SUPPLY9" gate="G$1" x="182.88" y="104.14" smashed="yes">
+<attribute name="VALUE" x="181.61" y="102.616" size="1.016" layer="96" align="top-left"/>
+</instance>
+<instance part="SUPPLY10" gate="GND" x="193.04" y="104.14" smashed="yes">
+<attribute name="VALUE" x="191.77" y="101.6" size="1.016" layer="96"/>
+</instance>
+<instance part="FB1" gate="G$1" x="187.96" y="106.68" smashed="yes" rot="R90">
+<attribute name="NAME" x="191.77" y="103.505" size="1.778" layer="95" rot="MR0"/>
+<attribute name="VALUE" x="191.77" y="109.855" size="1.778" layer="96" rot="R180"/>
+</instance>
 </instances>
 <busses>
 </busses>
 <nets>
+<net name="VDD" class="0">
+<segment>
+<pinref part="C1" gate="G$1" pin="2"/>
+<pinref part="C2" gate="G$1" pin="2"/>
+<wire x1="63.5" y1="132.08" x2="55.88" y2="132.08" width="0.1524" layer="91"/>
+<label x="58.42" y="132.08" size="1.778" layer="95"/>
+</segment>
+<segment>
+<pinref part="U5" gate="A" pin="DVDD"/>
+<wire x1="91.44" y1="127" x2="78.74" y2="127" width="0.1524" layer="91"/>
+<wire x1="78.74" y1="127" x2="78.74" y2="134.62" width="0.1524" layer="91"/>
+<label x="78.74" y="134.62" size="1.778" layer="95"/>
+</segment>
+<segment>
+<pinref part="U5" gate="A" pin="AVDD1"/>
+<pinref part="U5" gate="A" pin="AVDD2"/>
+<wire x1="91.44" y1="132.08" x2="91.44" y2="129.54" width="0.1524" layer="91"/>
+<wire x1="91.44" y1="129.54" x2="83.82" y2="129.54" width="0.1524" layer="91"/>
+<wire x1="83.82" y1="129.54" x2="83.82" y2="134.62" width="0.1524" layer="91"/>
+<label x="83.82" y="134.62" size="1.778" layer="95"/>
+</segment>
+<segment>
+<pinref part="R2" gate="G$1" pin="2"/>
+<wire x1="149.86" y1="119.38" x2="152.4" y2="119.38" width="0.1524" layer="91"/>
+<pinref part="R3" gate="G$1" pin="2"/>
+<wire x1="152.4" y1="119.38" x2="157.48" y2="119.38" width="0.1524" layer="91"/>
+<wire x1="157.48" y1="119.38" x2="157.48" y2="116.84" width="0.1524" layer="91"/>
+<wire x1="152.4" y1="119.38" x2="152.4" y2="121.92" width="0.1524" layer="91"/>
+<label x="152.4" y="121.92" size="1.778" layer="95"/>
+</segment>
+<segment>
+<pinref part="U6" gate="A" pin="VDD"/>
+<wire x1="88.9" y1="73.66" x2="83.82" y2="73.66" width="0.1524" layer="91"/>
+<wire x1="83.82" y1="73.66" x2="83.82" y2="76.2" width="0.1524" layer="91"/>
+<label x="83.82" y="76.2" size="1.778" layer="95"/>
+</segment>
+</net>
+<net name="GND" class="0">
+<segment>
+<pinref part="C2" gate="G$1" pin="1"/>
+<pinref part="C1" gate="G$1" pin="1"/>
+<wire x1="55.88" y1="127" x2="63.5" y2="127" width="0.1524" layer="91"/>
+<pinref part="SUPPLY6" gate="GND" pin="GND"/>
+<junction x="55.88" y="127"/>
+</segment>
+<segment>
+<pinref part="U5" gate="A" pin="DGND"/>
+<pinref part="SUPPLY8" gate="GND" pin="GND"/>
+<wire x1="134.62" y1="121.92" x2="132.08" y2="121.92" width="0.1524" layer="91"/>
+</segment>
+<segment>
+<pinref part="FB1" gate="G$1" pin="P$2"/>
+<pinref part="SUPPLY10" gate="GND" pin="GND"/>
+<wire x1="190.5" y1="106.68" x2="193.04" y2="106.68" width="0.1524" layer="91"/>
+</segment>
+</net>
+<net name="SDA" class="0">
+<segment>
+<pinref part="U5" gate="A" pin="SDA"/>
+<pinref part="R2" gate="G$1" pin="1"/>
+<wire x1="132.08" y1="111.76" x2="149.86" y2="111.76" width="0.1524" layer="91"/>
+<label x="137.16" y="111.76" size="1.778" layer="95"/>
+</segment>
+<segment>
+<pinref part="J6" gate="G$1" pin="1"/>
+<wire x1="142.24" y1="99.06" x2="149.86" y2="99.06" width="0.1524" layer="91"/>
+<label x="147.32" y="99.06" size="1.778" layer="95"/>
+</segment>
+</net>
+<net name="SCL" class="0">
+<segment>
+<pinref part="U5" gate="A" pin="SCL"/>
+<pinref part="R3" gate="G$1" pin="1"/>
+<wire x1="132.08" y1="109.22" x2="157.48" y2="109.22" width="0.1524" layer="91"/>
+<label x="137.16" y="109.22" size="1.778" layer="95"/>
+</segment>
+<segment>
+<pinref part="J6" gate="G$1" pin="2"/>
+<wire x1="142.24" y1="101.6" x2="149.86" y2="101.6" width="0.1524" layer="91"/>
+<label x="147.32" y="101.6" size="1.778" layer="95"/>
+</segment>
+</net>
+<net name="AGND" class="0">
+<segment>
+<pinref part="U5" gate="A" pin="AGND2"/>
+<pinref part="U5" gate="A" pin="AGND1"/>
+<wire x1="132.08" y1="119.38" x2="132.08" y2="116.84" width="0.1524" layer="91"/>
+<wire x1="132.08" y1="116.84" x2="134.62" y2="116.84" width="0.1524" layer="91"/>
+<pinref part="SUPPLY7" gate="G$1" pin="AGND"/>
+</segment>
+<segment>
+<pinref part="SUPPLY9" gate="G$1" pin="AGND"/>
+<pinref part="FB1" gate="G$1" pin="P$1"/>
+<wire x1="182.88" y1="106.68" x2="185.42" y2="106.68" width="0.1524" layer="91"/>
+</segment>
+</net>
+<net name="VIN" class="0">
+<segment>
+<pinref part="U5" gate="A" pin="VIN"/>
+<wire x1="91.44" y1="121.92" x2="78.74" y2="121.92" width="0.1524" layer="91"/>
+<wire x1="78.74" y1="121.92" x2="78.74" y2="109.22" width="0.1524" layer="91"/>
+<label x="83.82" y="121.92" size="1.778" layer="95"/>
+<pinref part="RFB" gate="G$1" pin="1"/>
+<wire x1="81.28" y1="109.22" x2="78.74" y2="109.22" width="0.1524" layer="91"/>
+</segment>
+</net>
+<net name="VOUT" class="0">
+<segment>
+<pinref part="U5" gate="A" pin="VOUT"/>
+<wire x1="91.44" y1="119.38" x2="86.36" y2="119.38" width="0.1524" layer="91"/>
+<label x="83.82" y="119.38" size="1.778" layer="95"/>
+</segment>
+</net>
+<net name="N$2" class="0">
+<segment>
+<pinref part="RFB" gate="G$1" pin="2"/>
+<pinref part="U5" gate="A" pin="RFB"/>
+<wire x1="88.9" y1="109.22" x2="91.44" y2="109.22" width="0.1524" layer="91"/>
+</segment>
+</net>
 </nets>
 </sheet>

Commit message: finish up test board
Parts:
- added C3, C4: 1uF, scono:CAP0603-CAP
- added J7: SEL, scono:CONN_02
- added R4: 510K, scono:R-US_R0603
- added R5: 200K, scono:R-US_R0603
- added R6: 100K, scono:R-US_R0603
- R2, R3: value (none) -> 10K
- renumbered U$1 to D1
Connections:
- new net N$10: C3.2, U6.S3B
- new net N$11: C4.1, R6.1, U6.S4A
- new net N$12: C4.2, R6.2, U6.S4B
- new net N$3: J7.1, U6.A1
- new net N$4: J7.2, U6.A0
- new net N$5: R4.2, U6.S1A
- new net N$6: R4.1, U6.S1B
- new net N$7: R5.2, U6.S2A
- new net N$8: R5.1, U6.S2B
- new net N$9: C3.1, U6.S3A
- net GND: now also U6.GND, U6.VSS
- net VDD: now also U6.EN
- net VIN: now also U6.DA
- net VOUT: now also U6.DB

Commit message: finalize prototype
Parts:
- added C5: 0.1uF, scono:CAP0603-CAP
- added C6: 10uF, scono:CAP0603-CAP
- J6: value SDA -> I2C
- U5: value AD5933YRSZ -> AD5933
Connections:
- net GND: now also C5.1, C6.1
- net VDD: now also C5.2, C6.2
Changed lines of the file:
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@@
 <attribute name="SUBSYSTEM_NAME" value="Imepdence"/>
 </part>
-<part name="U5" library="scono" deviceset="AD5933YRSZ" device=""/>
+<part name="U5" library="scono" deviceset="AD5933YRSZ" device="" value="AD5933"/>
 <part name="C1" library="scono" deviceset="CAP" device="0603-CAP" value="0.1uF"/>
 <part name="C2" library="scono" deviceset="CAP" device="0603-CAP" value="10uF"/>
@@
 <part name="SUPPLY7" library="scono" deviceset="AGND" device=""/>
 <part name="SUPPLY8" library="scono" deviceset="GND" device=""/>
-<part name="J6" library="scono" deviceset="CONN_02" device="" package3d_urn="urn:adsk.eagle:package:38039/1" value="SDA"/>
+<part name="J6" library="scono" deviceset="CONN_02" device="" package3d_urn="urn:adsk.eagle:package:38039/1" value="I2C"/>
 <part name="RFB" library="scono" deviceset="R-US_" device="R0603" value="1M"/>
 <part name="U6" library="scono" deviceset="ADG1609" device=""/>
@@
 <part name="R6" library="scono" deviceset="R-US_" device="R0603" value="100K"/>
 <part name="U1" library="scono" deviceset="LM334Z/NOPB" device=""/>
+<part name="C5" library="scono" deviceset="CAP" device="0603-CAP" value="0.1uF"/>
+<part name="C6" library="scono" deviceset="CAP" device="0603-CAP" value="10uF"/>
+<part name="SUPPLY13" library="scono" deviceset="GND" device=""/>
 </parts>
 <sheets>
@@
 <attribute name="VALUE" x="72.39" y="50.8" size="1.016" layer="96" rot="R270" align="top-left"/>
 </instance>
+<instance part="C5" gate="G$1" x="66.04" y="73.66" smashed="yes" rot="R90">
+<attribute name="NAME" x="64.516" y="72.39" size="1.016" layer="95" rot="R90"/>
+<attribute name="VALUE" x="68.58" y="72.39" size="1.016" layer="96" rot="R90"/>
+</instance>
+<instance part="C6" gate="G$1" x="58.42" y="73.66" smashed="yes" rot="R90">
+<attribute name="NAME" x="56.896" y="72.39" size="1.016" layer="95" rot="R90"/>
+<attribute name="VALUE" x="60.96" y="72.39" size="1.016" layer="96" rot="R90"/>
+</instance>
+<instance part="SUPPLY13" gate="GND" x="58.42" y="68.58" smashed="yes">
+<attribute name="VALUE" x="57.15" y="66.04" size="1.016" layer="96"/>
+</instance>
 </instances>
 <busses>
@@
 <label x="144.78" y="66.04" size="1.778" layer="95"/>
 </segment>
+<segment>
+<pinref part="C5" gate="G$1" pin="2"/>
+<pinref part="C6" gate="G$1" pin="2"/>
+<wire x1="66.04" y1="76.2" x2="58.42" y2="76.2" width="0.1524" layer="91"/>
+<label x="60.96" y="76.2" size="1.778" layer="95"/>
+</segment>
 </net>
 <net name="GND" class="0">
@@
 <pinref part="SUPPLY12" gate="GND" pin="GND"/>
 </segment>
-</net>
+<segment>
+<pinref part="C6" gate="G$1" pin="1"/>
+<pinref part="C5" gate="G$1" pin="1"/>
+<wire x1="58.42" y1="71.12" x2="66.04" y2="71.12" width="0.1524" layer="91"/>
+<pinref part="SUPPLY13" gate="GND" pin="GND"/>
+<junction x="58.42" y="71.12"/>
+</segment>
+</net>
