File: oximeter/oximeter.sch (EAGLE design)
At the start: 24 parts, among them U1 AFE4490_AFE4490, U2 AZ1117EH-3.3TRG1, X1 FFC-32

Commit message: more nextflex progress
Parts:
- removed X1: FFC-32, scono:FFC-32
- added J3: FFC-32, scono:FFC-32
Connections:
- new net N$1: J3.31
- new net N$2: J3.15
- new net N$3: J3.27
- new net N$4: J3.11
- new net N$8: J3.19
- new net N$9: J3.23
- net INN: now also J3.20; no longer X1-13.1, X1-14.1
- net INP: now also J3.24; no longer X1-10.1, X1-9.1
- net TXN: now also J3.16, J3.32; no longer X1-1.1, X1-17.1, X1-18.1, X1-2.1
- net TXP: now also J3.12, J3.28; no longer X1-21.1, X1-22.1, X1-5.1, X1-6.1
