File: NextFlex/nextflex_revb.brd (EAGLE design)
At the start: 54.5 x 79 mm, 72 parts, among them J1 FFC-32, J2 USB, J4 BAT, J5 FFC-32, J8 BURNIN, SW1 BTN-PTS810, U1 DG406DYZ-T, U2 DG406DYZ-T, U3 AD5933YRSZ, U4 AFE4490_AFE4490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

Commit message: place final revision order for next flex
Routing:
- net SDA: track 54.0 -> 46.1 mm, vias 1 -> 0
- net GND: track 181.3 -> 186.2 mm, vias 26 -> 27
- net 5V: track 92.9 -> 97.6 mm
- net MUX_2_SEL_1: track 88.3 -> 90.2 mm
Changed lines of the file:
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@@
 <wire x1="19.75" y1="71.1" x2="19.75" y2="72.623" width="0.254" layer="1"/>
 <wire x1="19.75" y1="72.623" x2="19.877" y2="72.75" width="0.254" layer="1"/>
-<wire x1="19.75" y1="71.1" x2="19.6" y2="71.25" width="0.254" layer="1"/>
 <wire x1="44.57564375" y1="37.674353125" x2="45.075646875" y2="37.674353125" width="0.508" layer="1"/>
 <wire x1="45.075646875" y1="37.674353125" x2="47" y2="35.75" width="0.508" layer="1"/>
@@
 <wire x1="16.7" y1="62.7" x2="17.75" y2="63.75" width="0.1524" layer="1"/>
 <via x="17.75" y="63.75" extent="1-16" drill="0.39"/>
-<wire x1="36" y1="53.5" x2="36" y2="55.75" width="0" layer="19" extent="1-1"/>
+<wire x1="36" y1="55.75" x2="36" y2="53.5" width="0.1524" layer="16"/>
+<wire x1="36" y1="55.75" x2="36" y2="57.25" width="0.1524" layer="1"/>
+<wire x1="36" y1="57.25" x2="37" y2="58.25" width="0.1524" layer="1"/>
+<via x="37" y="58.25" extent="1-16" drill="0.4"/>
 </signal>
 <signal name="E1">
@@
 <wire x1="30.93025" y1="57.1339" x2="31.055590625" y2="57.259240625" width="0.1524" layer="1"/>
 <wire x1="31.055590625" y1="57.259240625" x2="32.009240625" y2="57.259240625" width="0.1524" layer="1"/>
-<wire x1="32.25" y1="55.75" x2="32.25" y2="57.25" width="0.1524" layer="16"/>
+<wire x1="32.25" y1="55.75" x2="32.25" y2="56.75" width="0.1524" layer="16"/>
 <wire x1="37" y1="51" x2="32.25" y2="55.75" width="0.1524" layer="16"/>
 <wire x1="37" y1="44.5" x2="37" y2="51" width="0.1524" layer="16"/>
@@
 <wire x1="27.25" y1="20.5" x2="29.25" y2="22.5" width="0.1524" layer="16"/>
 <wire x1="27.25" y1="19" x2="27.25" y2="20.5" width="0.1524" layer="16"/>
-<wire x1="32.25" y1="57.25" x2="32.009240625" y2="57.259240625" width="0.1524" layer="16"/>
+<wire x1="32.009240625" y1="57.259240625" x2="32.25" y2="57.01848125" width="0.1524" layer="16"/>
+<wire x1="32.25" y1="57.01848125" x2="32.25" y2="56.75" width="0.1524" layer="16"/>
 </signal>
 <signal name="MUX_2_SEL_1">
@@
 <wire x1="30.65074375" y1="56.37425625" x2="31.62425625" y2="56.37425625" width="0.1524" layer="1"/>
 <via x="31.62425625" y="56.37425625" extent="1-16" drill="0.39"/>
-<wire x1="31.5" y1="56.75" x2="31.5" y2="56.5" width="0.1524" layer="16"/>
-<wire x1="31.25" y1="57" x2="31.5" y2="56.75" width="0.1524" layer="16"/>
+<wire x1="31.5" y1="56.75" x2="31.25" y2="57" width="0.1524" layer="16"/>
 <wire x1="31.25" y1="57.5" x2="31.25" y2="57" width="0.1524" layer="16"/>
-<wire x1="31.75" y1="58" x2="31.25" y2="57.5" width="0.1524" layer="16"/>
-<wire x1="32.5" y1="58" x2="31.75" y2="58" width="0.1524" layer="16"/>
-<wire x1="40" y1="50.5" x2="32.5" y2="58" width="0.1524" layer="16"/>
-<wire x1="40" y1="45.25" x2="40" y2="50.5" width="0.1524" layer="16"/>
+<wire x1="31.25" y1="57.5" x2="31.75" y2="58" width="0.1524" layer="16"/>
+<wire x1="40" y1="50.5" x2="40" y2="45.25" width="0.1524" layer="16"/>
 <wire x1="43.5" y1="41.75" x2="40" y2="45.25" width="0.1524" layer="16"/>
 <wire x1="43.5" y1="39.75" x2="43.5" y2="41.75" width="0.1524" layer="16"/>
@@
 <wire x1="28.5" y1="21.25" x2="29.75" y2="22.5" width="0.1524" layer="16"/>
 <wire x1="28.5" y1="19" x2="28.5" y2="21.25" width="0.1524" layer="16"/>
-<wire x1="31.5" y1="56.5" x2="31.62425625" y2="56.37425625" width="0.1524" layer="16"/>
+<wire x1="35.75" y1="58" x2="38" y2="55.75" width="0.1524" layer="16"/>
+<wire x1="38" y1="55.75" x2="38" y2="52.5" width="0.1524" layer="16"/>
+<wire x1="38" y1="52.5" x2="40" y2="50.5" width="0.1524" layer="16"/>
+<wire x1="31.75" y1="58" x2="35.75" y2="58" width="0.1524" layer="16"/>
+<wire x1="31.62425625" y1="56.37425625" x2="31.5" y2="56.4985125" width="0.1524" layer="16"/>
+<wire x1="31.5" y1="56.4985125" x2="31.5" y2="56.75" width="0.1524" layer="16"/>
 </signal>
 <signal name="MUX_2_SEL_2">
@@
 <wire x1="8.1" y1="32.75" x2="16.5" y2="32.75" width="0.1524" layer="1"/>
 <contactref element="U8" pad="19"/>
-<via x="21.75" y="54.398" extent="1-16" drill="0.39"/>
 <wire x1="23.975" y1="56" x2="23.8411" y2="55.8661" width="0.1524" layer="1"/>
 <wire x1="23.8411" y1="55.8661" x2="23.56975" y2="55.8661" width="0.1524" layer="1"/>
-<wire x1="22.10165" y1="54.398" x2="21.75" y2="54.398" width="0.1524" layer="1"/>
 <wire x1="23.56975" y1="55.8661" x2="22.10165" y2="54.398" width="0.1524" layer="1"/>
-<wire x1="21.75" y1="54.398" x2="21.75" y2="55.25" width="0.1524" layer="16"/>
-<wire x1="21.75" y1="55.25" x2="23.75" y2="57.25" width="0.1524" layer="16"/>
-<wire x1="23.75" y1="57.25" x2="23.75" y2="58.25" width="0.1524" layer="16"/>
-<wire x1="23.75" y1="58.25" x2="22" y2="60" width="0.1524" layer="16"/>
-<wire x1="22" y1="60" x2="21.25" y2="60" width="0.1524" layer="16"/>
-<wire x1="21.75" y1="54.398" x2="17.398" y2="54.398" width="0.1524" layer="1"/>
 <wire x1="16" y1="47.5" x2="8.75" y2="40.25" width="0.1524" layer="1"/>
 <wire x1="17.398" y1="54.398" x2="16" y2="53" width="0.1524" layer="1"/>
 <wire x1="16" y1="53" x2="16" y2="47.5" width="0.1524" layer="1"/>
+<wire x1="22.10165" y1="54.398" x2="17.398" y2="54.398" width="0.1524" layer="1"/>
 </signal>
 <signal name="SCL">
@@
 <wire x1="32.012" y1="77.238" x2="33.5" y2="75.75" width="0.254" layer="16"/>
 <wire x1="21.988" y1="77.238" x2="32.012" y2="77.238" width="0.254" layer="16"/>
-<wire x1="33.92" y1="49.79" x2="31.25" y2="53" width="0" layer="19" extent="1-1"/>
+<wire x1="31.25" y1="53" x2="32.24989375" y2="52.00010625" width="0.254" layer="16"/>
+<wire x1="32.24989375" y1="52.00010625" x2="32.24989375" y2="51.40190625" width="0.254" layer="16"/>
+<wire x1="32.24989375" y1="51.40190625" x2="32.6889125" y2="50.9628875" width="0.254" layer="16"/>
+<wire x1="32.6889125" y1="50.9628875" x2="33.33084375" y2="50.9628875" width="0.254" layer="16"/>
+<wire x1="33.33084375" y1="50.9628875" x2="33.92" y2="50.37373125" width="0.254" layer="16"/>
+<wire x1="33.92" y1="50.37373125" x2="33.92" y2="49.79" width="0.254" layer="16"/>
 </signal>
 <signal name="N$16">
@@
 <contactref element="U7" pad="10"/>
 <contactref element="J6" pad="4"/>
-<wire x1="33.5" y1="51.070665625" x2="33.570665625" y2="51.070665625" width="0.1524" layer="1"/>
 <wire x1="37.4" y1="36.3194" x2="37.4" y2="37.4" width="0.1524" layer="1"/>
 <wire x1="41.23236875" y1="40.25" x2="42.12" y2="40.25" width="0.1524" layer="1"/>
